Commit message: t800: align delivery knee limits

File: assets/resource/robot/t800/urdf/serial_t800.urdf (robot description, URDF)
Before this commit: robot t800, 30 links, 29 joints
Joints:
- joint J03_KNEE_PITCH_L: limit lower=0.0 upper=2.355 effort=415 velocity=25.96 -> lower=-0.261667 upper=2.355 effort=415 velocity=25.96
- joint J09_KNEE_PITCH_R: limit lower=0.0 upper=2.355 effort=415 velocity=25.96 -> lower=-0.261667 upper=2.355 effort=415 velocity=25.96
